File: left.kicad_sch (KiCad schematic)
At the start: 43 parts, among them J2 OLED_128x32, SW2 Switch, U2 Nice_Nano_V2

Commit message: Formato de teclado listo
Parts:
- renumbered D25 to D21, D24 to D22, D22 to D24, D21 to D25, D30 to D26, D29 to D27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
