File: custom.kicad_pcb (KiCad board)
At the start: 2 copper layers, 285.7 x 93.9 mm, 86 parts, among them J1 OLED_128x32, J2 OLED_128x32, SW1 Switch, SW2 Switch, U1 Nice_Nano_V2, U2 Nice_Nano_V2

Commit message: Formato de teclado listo
Parts:
- removed SW1, SW2: Switch, Button_Switch_SMD:SW_Push_1P1T_NO_Vertical_Wuerth_434133025816
- added KY2: Switch, Button_Switch_SMD:SW_Push_1P1T_NO_Vertical_Wuerth_434133025816, F.Cu at (-75.7, -42.7)
- added KY3: Switch, Button_Switch_SMD:SW_Push_1P1T_NO_Vertical_Wuerth_434133025816, F.Cu at (-13.9, 89.2)
- D1, D10, D11, D12, D13, D14, D15, D16, D17, D18, D19, D2, D20, D21, D22, D23, D24, D25, D26, D27, D28, D29, D3, D30, D31, D32, D33, D34, D35, D36, D37, D38, D39, D4, D40, D5, D6, D7, D8, D9, MX1, MX10, MX11, MX12, MX13, MX14, MX15, MX16, MX17, MX18, MX19, MX2, MX21, MX22, MX23, MX24, MX25, MX26, MX27, MX28, MX29, MX3, MX30, MX31, MX32, MX33, MX34, MX35, MX38, MX39, MX4, MX5, MX6, MX7, MX8, MX9: moved to F.Cu
- MX20, MX40: footprint PCM_marbastlib-mx:SW_MX_HS_CPG151101S11_1.25u -> PCM_marbastlib-mx:SW_MX_HS_CPG151101S11_1u; moved to F.Cu
- MX36, MX37: footprint PCM_marbastlib-mx:SW_MX_HS_CPG151101S11_1u -> PCM_marbastlib-mx:SW_MX_HS_CPG151101S11_1.25u; moved to F.Cu
- moved D26 392.2 mm to (-94.8, 44.7)
- moved D21 379.8 mm to (-84.7, 50.5)
- moved D31 378.7 mm to (-78.0, 44.7)
- moved D27 368.6 mm to (-91.4, 44.7)
- moved D33 359.4 mm to (-98.1, 39.0)
- moved D22 356.1 mm to (-81.4, 50.5)
- moved D32 355.3 mm to (-74.7, 44.7)
- moved D37 351.0 mm to (-84.7, 39.0)
- moved D28 345.1 mm to (-88.1, 44.7)
- moved D34 336.0 mm to (-94.8, 39.0)
- moved D23 332.5 mm to (-78.0, 50.5)
- moved D38 327.2 mm to (-81.4, 39.0)
- moved D25 324.5 mm to (-98.1, 44.7)
- moved D29 320.5 mm to (-84.7, 44.7)
- moved D39 316.4 mm to (-78.0, 39.0), turned to 90 degrees
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Connections:
- D10 pad 1: ROW 2 -> ROW 1-R
- D11 pad 1: ROW 3 -> ROW 2
- D12 pad 1: ROW 3 -> ROW 2
- D13 pad 1: ROW 3 -> ROW 2
- D14 pad 1: ROW 3 -> ROW 2
- D15 pad 1: ROW 3 -> ROW 2
- D16 pad 1: ROW 3 -> ROW 2-R
- D17 pad 1: ROW 4 -> ROW 2-R
- D18 pad 1: ROW 4 -> ROW 2-R
- D19 pad 1: ROW 4 -> ROW 2-R
- D20 pad 1: ROW 4 -> ROW 2-R
- D21 pad 1: ROW 1-R -> ROW 3
- D22 pad 1: ROW 1-R -> ROW 3
- D23 pad 1: ROW 1-R -> ROW 3
- D24 pad 1: ROW 1-R -> ROW 3
- D25 pad 1: ROW 1-R -> ROW 3
- D26 pad 1: ROW 2-R -> ROW 3
- D27 pad 1: ROW 2-R -> ROW 3-R
- D28 pad 1: ROW 2-R -> ROW 3-R
- D29 pad 1: ROW 2-R -> ROW 3-R
- D30 pad 1: ROW 2-R -> ROW 3-R
- D33 pad 1: ROW 3-R -> ROW 4
- D34 pad 1: ROW 3-R -> ROW 4
- D35 pad 1: ROW 3-R -> ROW 4
- D36 pad 1: ROW 3-R -> ROW 4
- D6 pad 1: ROW 2 -> ROW 1-R
- D7 pad 1: ROW 2 -> ROW 1-R
- D8 pad 1: ROW 2 -> ROW 1-R
- D9 pad 1: ROW 2 -> ROW 1-R
- MX10 pad 1: COL 5 -> COL 1-R
- MX16 pad 1: COL 6 -> COL 5-R
- MX17 pad 1: COL 3 -> COL 4-R
- MX18 pad 1: COL 4 -> COL 3-R
- MX19 pad 1: COL 5 -> COL 2-R
- MX20 pad 1: COL 6 -> COL 1-R
- MX21 pad 1: COL 1-R -> COL 1
- MX22 pad 1: COL 2-R -> COL 2
- MX23 pad 1: COL 3-R -> COL 3
- MX24 pad 1: COL 4-R -> COL 4
- MX25 pad 1: COL 5-R -> COL 5
- MX26 pad 1: COL 1-R -> COL 6
- MX27 pad 1: COL 2-R -> COL 6-R
- MX28 pad 1: COL 3-R -> COL 5-R
- MX30 pad 1: COL 5-R -> COL 3-R
- MX31 pad 1: COL 1-R -> COL 2-R
- MX32 pad 1: COL 2-R -> COL 1-R
- MX33 pad 1: COL 3-R -> COL 3
- MX34 pad 1: COL 4-R -> COL 4
- MX35 pad 1: COL 5-R -> COL 5
- MX36 pad 1: COL 6-R -> COL 6
- MX37 pad 1: COL 3-R -> COL 6-R
- MX38 pad 1: COL 4-R -> COL 5-R
- MX39 pad 1: COL 5-R -> COL 4-R
- MX40 pad 1: COL 6-R -> COL 3-R
- MX6 pad 1: COL 1 -> COL 5-R
- MX7 pad 1: COL 2 -> COL 4-R
- MX8 pad 1: COL 3 -> COL 3-R
- MX9 pad 1: COL 4 -> COL 2-R
Routing:
- net COL 1: track 167.7 -> 0.00 mm, vias 1 -> 0
- net COL 3: track 161.2 -> 0.00 mm, vias 4 -> 0
- net COL 2: track 156.0 -> 0.00 mm, vias 3 -> 0
- net COL 4: track 143.7 -> 0.00 mm, vias 4 -> 0
- net ROW 3: track 130.8 -> 0.00 mm
- net COL 5: track 127.2 -> 0.00 mm, vias 4 -> 0
- net ROW 1: track 108.6 -> 0.00 mm
- net ROW 2: track 107.4 -> 0.00 mm
- net ROW 4: track 103.4 -> 0.00 mm
- net ROW 3-R: track 92.3 -> 0.00 mm
- net GND-R: track 70.4 -> 0.00 mm, vias 1 -> 0
- net ROW 1-R: track 70.0 -> 0.00 mm
- net ROW 2-R: track 70.0 -> 0.00 mm
- net GND: track 68.0 -> 0.00 mm
- net ROW 4-R: track 52.3 -> 0.00 mm
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Other:
- board outline removed

Commit message: Se colocan diodos
Parts:
- moved D10 416.7 mm to (321.7, 42.9)
- moved D20 410.0 mm to (321.7, 62.9)
- moved D9 400.1 mm to (301.7, 41.2)
- moved D32 398.2 mm to (321.7, 82.9)
- moved D19 393.3 mm to (301.7, 61.2)
- moved D31 381.5 mm to (301.7, 81.2)
- moved D18 376.6 mm to (281.7, 60.0)
- moved D30 364.8 mm to (281.7, 80.0)
- moved D40 361.6 mm to (281.7, 100.3)
- moved D17 360.0 mm to (261.7, 61.2)
- moved D8 357.1 mm to (281.7, 40.0)
- moved D29 348.3 mm to (261.7, 81.2)
- moved D39 345.4 mm to (261.7, 101.4)
- moved D6 340.4 mm to (258.4, 41.2)
- moved D7 340.4 mm to (261.7, 41.2)
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